File: hardware/geoBit.kicad_pcb (KiCad board)
At the start: 4 copper layers, 60 x 55 mm, 91 parts, among them CN2 ATGM336H-6N-74, CN4 S2B-PH-SM4-TB(LF)(SN), J1 Conn_01x03_Pin, Q3 Si1308EDL, Q4 JSM2302, SW2 SW_Push, SW4 ON/OFF, SW61 K2-1103ST-A4SW-04, SW62 K2-1103ST-A4SW-04, SW63 K2-1103ST-A4SW-04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

Commit message: Updated pcb v0.1
Parts:
- removed C44, C45: 10uF, Capacitor_SMD:C_0603_1608Metric_Pad1.08x0.95mm_HandSolder
- removed CARD1: MT102010052, easyeda2kicad:TF-CARD-SMD_MT102010052
- removed R45: 1M, Resistor_SMD:R_0402_1005Metric_Pad0.72x0.64mm_HandSolder
- removed R46: 2R, Resistor_SMD:R_0402_1005Metric
- removed USBC4: 105450-0101, easyeda2kicad:USB-C-SMD_TYPE-C-USB-18
- added C19: 10uF, Capacitor_SMD:C_0603_1608Metric_Pad1.08x0.95mm_HandSolder, F.Cu at (107.4, 49.2)
- added C20: 10uF, Capacitor_SMD:C_0603_1608Metric_Pad1.08x0.95mm_HandSolder, F.Cu at (109.1, 49.1)
- added R7: 1M, Resistor_SMD:R_0402_1005Metric_Pad0.72x0.64mm_HandSolder, F.Cu at (95.1, 54.6)
- added R9: 2R, Resistor_SMD:R_0402_1005Metric, F.Cu at (109.1, 51.8)
- added U3: MR01A-01239, easyeda2kicad:TF-SMD_MR01A-01211, F.Cu at (85.7, 70.3)
- added USB1: TYPE-C 16PIN 2MD(073), easyeda2kicad:USB-C-SMD_TYPE-C-6PIN-2MD-073, F.Cu at (101.2, 52.0)
- CN2: footprint ATGM336H:ATGM336H-5N31 -> EasyEDA:COMM-SMD_18P-L10.1-W9.7-P1.1-TL_L76-LB
- J1: value Conn_01x03_Pin -> Conn_01x12_Pin; footprint Connector_PinHeader_2.54mm:PinHeader_1x03_P2.54mm_Vertical -> Connector_PinSocket_2.54mm:PinSocket_1x12_P2.54mm_Vertical
- moved R61 20.6 mm to (91.2, 57.0), turned to 180 degrees
- moved C50 14.8 mm to (93.2, 85.0), turned to 180 degrees
- moved R63 14.4 mm to (108.0, 85.2)
- moved U5 11.0 mm to (95.2, 72.4), turned to 0 degrees
- moved J1 9.06 mm to (105.7, 92.3), turned to 90 degrees
- moved C9 8.89 mm to (100.2, 85.4)
- moved R62 5.40 mm to (93.7, 82.8), turned to 180 degrees
- moved C12 5.11 mm to (97.6, 69.1), turned to 90 degrees
- moved C8 4.02 mm to (101.4, 85.3)
- moved C7 2.57 mm to (95.9, 76.9)
- moved C3 2.49 mm to (110.8, 69.4)
- moved C4 2.41 mm to (112.0, 69.4)
- moved C6 2.33 mm to (99.8, 69.1), turned to 90 degrees
- moved C11 1.98 mm to (109.8, 79.2)
- moved C10 1.45 mm to (112.5, 75.2)
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Connections:
- R43 pad 1: CC2 -> Net-(USB1-CC2)
- R44 pad 1: CC1 -> Net-(USB1-CC1)
- U1 pad 10: unconnected-(U1-GPIO7-Pad10) -> FILTERED_SD_DAT0
- U1 pad 12: unconnected-(U1-GPIO8-Pad12) -> FILTERED_SD_DAT1
- U1 pad 13: unconnected-(U1-GPIO9-Pad13) -> FILTERED_SD_DAT2
- U1 pad 14: unconnected-(U1-GPIO10-Pad14) -> FILTERED_SD_DAT3
- U1 pad 15: unconnected-(U1-GPIO11-Pad15) -> SD_DET
- U1 pad 16: unconnected-(U1-GPIO12-Pad16) -> GPS_RX
- U1 pad 17: unconnected-(U1-GPIO13-Pad17) -> GPS_TX
- U1 pad 18: unconnected-(U1-GPIO14-Pad18) -> GPS_1PPS
- U1 pad 19: unconnected-(U1-GPIO15-Pad19) -> STATUS_LED
- U1 pad 27: unconnected-(U1-GPIO16-Pad27) -> BUTTON3
- U1 pad 35: unconnected-(U1-GPIO23-Pad35) -> GPIO23
- U1 pad 36: unconnected-(U1-GPIO24-Pad36) -> GPIO24
- U1 pad 37: unconnected-(U1-GPIO25-Pad37) -> GPIO25
- U1 pad 40: unconnected-(U1-GPIO26_ADC0-Pad40) -> GPIO26_ADC0
- U1 pad 41: unconnected-(U1-GPIO27_ADC1-Pad41) -> GPIO27_ADC1
- U1 pad 42: unconnected-(U1-GPIO28_ADC2-Pad42) -> GPIO28_ADC2
- U1 pad 43: unconnected-(U1-GPIO29_ADC3-Pad43) -> GPIO29_ADC3
- U1 pad 5: STATUS_LED -> BUTTON1
- U1 pad 7: unconnected-(U1-GPIO4-Pad7) -> BUTTON2
- U1 pad 8: unconnected-(U1-GPIO5-Pad8) -> FILTERED_SD_CLK
- U1 pad 9: unconnected-(U1-GPIO6-Pad9) -> FILTERED_SD_CMD
- U5 pad 1: unconnected-(U5-WP/CD-Pad1) -> SD_DET
- U5 pad 10: FILTERED_SD_DAT1 -> SD_DAT1
- U5 pad 11: FILTERED_SD_DAT0 -> SD_DAT0
- U5 pad 12: FILTERED_SD_CLK -> SD_CLK
- U5 pad 13: FILTERED_SD_CMD -> SD_CMD
- U5 pad 14: FILTERED_SD_DAT3 -> SD_DAT3
- U5 pad 15: FILTERED_SD_DAT2 -> SD_DAT2
- U5 pad 3: SD_DAT2 -> FILTERED_SD_DAT2
- U5 pad 4: SD_DAT3 -> FILTERED_SD_DAT3
- U5 pad 5: SD_CMD -> FILTERED_SD_CMD
- U5 pad 6: SD_CLK -> FILTERED_SD_CLK
- U5 pad 7: SD_DAT0 -> FILTERED_SD_DAT0
- U5 pad 8: SD_DAT1 -> FILTERED_SD_DAT1
Routing:
- net GND: track 83.0 -> 193.3 mm, vias 24 -> 41
- net +3V3: track 108.1 -> 211.2 mm, vias 5 -> 10
- net GPIO29_ADC3: track 0.00 -> 45.5 mm, vias 0 -> 1
- net GPIO28_ADC2: track 0.00 -> 44.0 mm, vias 0 -> 1
- net GPIO27_ADC1: track 0.00 -> 43.9 mm, vias 0 -> 1
- net GPIO26_ADC0: track 0.00 -> 43.8 mm, vias 0 -> 1
- net BUTTON3: track 0.00 -> 43.1 mm, vias 0 -> 1
- net SD_DET: track 0.00 -> 34.6 mm, vias 0 -> 3
- net BUTTON2: track 3.73 -> 34.0 mm, vias 0 -> 3
- net GPIO25: track 0.00 -> 25.1 mm, vias 0 -> 1
- net GPIO24: track 0.00 -> 22.9 mm, vias 0 -> 1
- net Net-(USBC4-25): track 21.4 -> 0.00 mm
- net GPIO23: track 0.00 -> 21.1 mm, vias 0 -> 1
- net Net-(R7-Pad1): track 0.00 -> 19.0 mm, vias 0 -> 2
- net GPS_1PPS: track 1.66 -> 20.1 mm, vias 0 -> 2
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Other:
- board text added: "+"
- board text added: "-"
- board text added: "23"
- board text added: "24"
- board text added: "25"
- board text added: "26"
- board text added: "27"
- board text added: "28"
- board text added: "29"
- board text added: "3V3"
- board text added: "ADC"
- board text added: "Art by Snoof"
- board text added: "B1729"
- board text added: "BH6"
- board text added: "BOOT"
- board text added: "CLK"
- board text added: "DIO"
- board text added: "GND"
- board text added: "J5"
- board text added: "K9"
- board text added: "M42"
- board text added: "R2D2"
- board text added: "U7134"
- board text added: "Z101"
- board text added: "huffeec"
- board text added: "v0.1"
